File: hardware/prj-kicad/ethernet.kicad_sch (KiCad schematic)
At the start: 27 parts, among them J1 CONN_RJ45, Q1 BC846, T1 TRANSFORMER_1_1, U1 KSZ8091RN, X1 50MHz

Commit message: = UPD: Finish ESP32 routing (eth, boot, console, ...)
Parts:
- added R13: 10k, cowmotics-aquarea:SMD0603, symbol cowmotics-aquarea:R
- added TP5, TP6: CONN_1, cowmotics-aquarea:TP_SMD, symbol cowmotics-aquarea:CONN_1
Connections:
- net ETH_MDC: now also TP5.1
- net ETH_MDIO: now also TP6.1
- net GND: now also R13.1
- net CLK_EN renamed CLK50_EN
- net CLK50_EN: now also R13.2
Changed lines of the file:
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@@
+    (stroke (width 0) (type default) (color 0 0 0 0))
+  )
+  (wire (pts (xy 76.835 177.8) (xy 80.645 177.8))
     (stroke (width 0) (type default) (color 0 0 0 0))
   )
@@
     (stroke (width 0) (type default) (color 0 0 0 0))
   )
+  (wire (pts (xy 76.835 173.99) (xy 80.645 173.99))
+    (stroke (width 0) (type default) (color 0 0 0 0))
+  )
   (wire (pts (xy 36.195 143.51) (xy 36.195 144.78))
     (stroke (width 0) (type default) (color 0 0 0 0))
@@
     (stroke (width 0) (type default) (color 0 0 0 0))
   )
+  (wire (pts (xy 119.38 179.705) (xy 121.285 179.705))
+    (stroke (width 0) (type default) (color 0 0 0 0))
+  )
   (wire (pts (xy 134.62 58.42) (xy 142.24 58.42))
     (stroke (width 0) (type default) (color 0 0 0 0))
@@
     (stroke (width 0) (type default) (color 0 0 0 0))
   )
+  (wire (pts (xy 104.14 182.245) (xy 104.14 179.705))
+    (stroke (width 0) (type default) (color 0 0 0 0))
+  )
   (wire (pts (xy 129.54 71.12) (xy 129.54 58.42))
     (stroke (width 0) (type default) (color 0 0 0 0))
@@
   )
   (wire (pts (xy 36.195 158.75) (xy 36.195 160.02))
+    (stroke (width 0) (type default) (color 0 0 0 0))
+  )
+  (wire (pts (xy 104.14 179.705) (xy 106.68 179.705))
     (stroke (width 0) (type default) (color 0 0 0 0))
   )
@@
     )
   )
-  (global_label "CLK_EN" (shape input) (at 113.03 163.195 270) (fields_autoplaced)
-    (effects (font (size 1.016 1.016)) (justify right))
-    (property "Intersheet References" "${INTERSHEET_REFS}" (id 0) (at 112.9665 170.7376 90)
+  (global_label "CLK50_EN" (shape input) (at 113.03 163.195 270) (fields_autoplaced)
+    (effects (font (size 1.016 1.016)) (justify right))
+    (property "Intersheet References" "${INTERSHEET_REFS}" (id 0) (at 112.9665 172.6728 90)
       (effects (font (size 1.016 1.016)) (justify right) hide)
     )
@@
     )
   )
+  (global_label "CLK50_EN" (shape output) (at 121.285 179.705 0) (fields_autoplaced)
+    (effects (font (size 1.016 1.016)) (justify left))
+    (property "Intersheet References" "${INTERSHEET_REFS}" (id 0) (at 130.7628 179.6415 0)
+      (effects (font (size 1.016 1.016)) (justify left) hide)
+    )
+  )
+  (global_label "ETH_MDC" (shape input) (at 76.835 173.99 180) (fields_autoplaced)
+    (effects (font (size 1.016 1.016)) (justify right))
+    (property "Intersheet References" "${INTERSHEET_REFS}" (id 0) (at 68.1796 173.9265 0)
+      (effects (font (size 1.016 1.016)) (justify right) hide)
+    )
+  )
   (global_label "CLK_50M" (shape input) (at 101.6 120.65 180) (fields_autoplaced)
     (effects (font (size 1.016 1.016)) (justify right))
     (property "Intersheet References" "${INTERSHEET_REFS}" (id 0) (at 92.9446 120.5865 0)
+      (effects (font (size 1.016 1.016)) (justify right) hide)
+    )
+  )
+  (global_label "ETH_MDIO" (shape bidirectional) (at 76.835 177.8 180) (fields_autoplaced)
+    (effects (font (size 1.016 1.016)) (justify right))
+    (property "Intersheet References" "${INTERSHEET_REFS}" (id 0) (at 67.6475 177.7365 0)
       (effects (font (size 1.016 1.016)) (justify right) hide)
     )
@@
     (pin "1")
   )
+  (symbol (lib_id "cowmotics-aquarea:GND") (at 104.14 182.245 0) (unit 1)
+    (in_bom yes) (on_board yes) (fields_autoplaced)
+    (property "Reference" "#PWR0151" (id 0) (at 104.14 182.245 0)
+      (effects (font (size 0.762 0.762)) hide)
+    )
+    (property "Value" "GND" (id 1) (at 104.14 184.023 0)
+      (effects (font (size 0.762 0.762)) hide)
+    )
+    (property "Footprint" "" (id 2) (at 104.14 182.245 0)
+      (effects (font (size 1.524 1.524)))
+    )
+    (property "Datasheet" "" (id 3) (at 104.14 182.245 0)
+      (effects (font (size 1.524 1.524)))
+    )
+    (pin "1")
+  )
   (symbol (lib_id "cowmotics-aquarea:C") (at 142.24 64.77 0) (unit 1)
     (in_bom yes) (on_board yes)
@@
     (pin "2")
   )
+  (symbol (lib_id "cowmotics-aquarea:CONN_1") (at 84.455 173.99 0) (unit 1)
+    (in_bom yes) (on_board yes)
+    (property "Reference" "TP5" (id 0) (at 86.36 173.99 0)
+      (effects (font (size 1.016 1.016)) (justify left))
+    )
+    (property "Value" "CONN_1" (id 1) (at 84.455 172.593 0)
+      (effects (font (size 0.762 0.762)) hide)
+    )
+    (property "Footprint" "cowmotics-aquarea:TP_SMD" (id 2) (at 84.455 173.99 0)
+      (effects (font (size 1.524 1.524)) hide)
+    )
+    (property "Datasheet" "" (id 3) (at 84.455 173.99 0)
+      (effects (font (size 1.524 1.524)))
+    )
+    (pin "1")
+  )
   (symbol (lib_id "cowmotics-aquarea:GND") (at 121.92 115.57 0) (unit 1)
     (in_bom yes) (on_board yes) (fields_autoplaced)
@@
     (pin "10")
     (pin "11")
+    (pin "12")
+    (pin "13")
     (pin "14")
     (pin "15")
@@
     (pin "2")
     (pin "3")
+    (pin "4")
+    (pin "5")
     (pin "6")
     (pin "7")
@@
     (pin "9")
   )
+  (symbol (lib_id "cowmotics-aquarea:R") (at 113.03 179.705 90) (unit 1)
+    (in_bom yes) (on_board yes)
+    (property "Reference" "R13" (id 0) (at 113.03 177.165 90))
+    (property "Value" "10k" (id 1) (at 113.03 179.705 90)
+      (effects (font (size 1.016 1.016)))
+    )
+    (property "Footprint" "cowmotics-aquarea:SMD0603" (id 2) (at 113.03 179.705 0)
+      (effects (font (size 1.524 1.524)) hide)
+    )
+    (property "Datasheet" "" (id 3) (at 113.03 179.705 0)
+      (effects (font (size 1.524 1.524)))
+    )
+    (pin "1")
+    (pin "2")
+  )
   (symbol (lib_id "cowmotics-aquarea:OSC") (at 123.19 158.75 0) (unit 1)
     (in_bom yes) (on_board yes)
@@
     (pin "2")
   )
+  (symbol (lib_id "cowmotics-aquarea:CONN_1") (at 84.455 177.8 0) (unit 1)
+    (in_bom yes) (on_board yes)
+    (property "Reference" "TP6" (id 0) (at 86.36 177.8 0)
+      (effects (font (size 1.016 1.016)) (justify left))
+    )
+    (property "Value" "CONN_1" (id 1) (at 84.455 176.403 0)
+      (effects (font (size 0.762 0.762)) hide)
+    )
+    (property "Footprint" "cowmotics-aquarea:TP_SMD" (id 2) (at 84.455 177.8 0)
+      (effects (font (size 1.524 1.524)) hide)
+    )
+    (property "Datasheet" "" (id 3) (at 84.455 177.8 0)
+      (effects (font (size 1.524 1.524)))
+    )
+    (pin "1")
+  )
 )
