File: hardware/prj-kicad/mcu.kicad_sch (KiCad schematic)
At the start: 18 parts, among them U2 ESP32, U3 SST25VF016, X2 40MHz

Commit message: = UPD: Finish ESP32 routing (eth, boot, console, ...)
Parts:
- added C21: 100nF, cowmotics-aquarea:SMD0603, symbol cowmotics-aquarea:C
- added C22, C23: 1uF, cowmotics-aquarea:SMD0603, symbol cowmotics-aquarea:C
- added R17: 49.9, cowmotics-aquarea:SMD0603, symbol cowmotics-aquarea:R
- added R18: 0, cowmotics-aquarea:SMD0603, symbol cowmotics-aquarea:R
- added R19: 10k, cowmotics-aquarea:SMD0603, symbol cowmotics-aquarea:R
- added SW1: SW_PUSH, cowmotics-aquarea:SW_PTS840, symbol cowmotics-aquarea:SW_PUSH
- added SW2: SW_PUSH, cowmotics-aquarea:SW_434123043816, symbol cowmotics-aquarea:SW_PUSH
- added TP10, TP11, TP12, TP3, TP4, TP7, TP8, TP9: CONN_1, cowmotics-aquarea:TP_SMD, symbol cowmotics-aquarea:CONN_1
- A1: footprint (none) -> cowmotics-aquarea:CONN_SMA_RA
Connections:
- net +3.3V: now also C21.1
- net CLK_50M: now also R17.1; no longer U2.23 (GPIO0)
- net ETH_MDC: now also U2.34 (GPIO5)
- net ETH_MDIO: now also U2.36 (GPIO23)
- net ETH_RXER: now also R18.1; no longer U2.20 (MTCK)
- net GND: now also C21.2, C22.2, C23.2, R19.1, SW1.2, SW2.2, TP7.1
- net at R15.2, U2.9 (PU): now also C22.1, TP12.1
- net at U2.17 (MTMS): now also TP11.1
- net at U2.18 (MTDI): now also TP10.1
- net at U2.21 (MTDO): now also TP8.1
- net BOOT2: now reaches U2.22 (GPIO2)
- net BOOT2: now also R19.2
- net ETH_IRQ: now reaches U2.24 (GPIO4)
- net CLK50_EN: now reaches U2.35 (GPIO18)
- net U0_RX: now reaches U2.40 (U0_RX)
- net U0_RX: now also TP3.1
- net U0_TX: now reaches U2.41 (U0_TX)
- net U0_TX: now also TP4.1
- net RJ45_LED: now reaches U2.6 (SENSOR_CP)
- net BUTTON: now reaches U2.8 (SENSOR_VN)
- net BUTTON: now also C23.1, SW1.1
- new net: R18.2, TP9.1, U2.20 (MTCK)
- new net BOOT0: R17.2, SW2.1, U2.23 (GPIO0)
- no-connect marks 8 -> 6
